File: hardware/analog-in-v3.kicad_sch (KiCad schematic)
At the start: 31 parts

Commit message: Data Cleanup
Parts:
- C1: value (none) -> 10uF; footprint (none) -> kicad-libraries:C0805
- C2, C7: value (none) -> 100nF; footprint (none) -> kicad-libraries:C0603F
- C3: value (none) -> 180pF; footprint (none) -> kicad-libraries:C0603F
- C4: value (none) -> 15pF; footprint (none) -> kicad-libraries:C0603F
- C5: value (none) -> 220pF; footprint (none) -> kicad-libraries:C0402F
- C6: value (none) -> 1uF; footprint (none) -> kicad-libraries:C0603F
- D1: value (none) -> 3V3; footprint (none) -> kicad-libraries:MiniMelf
- D2: value (none) -> 5V; footprint (none) -> kicad-libraries:MiniMelf
- D3: value (none) -> blue; footprint (none) -> kicad-libraries:D0603F
- F1, F2: value (none) -> OZCJ0035FF2G; footprint (none) -> kicad-libraries:F1206
- P1: value (none) -> CON-SENSOR2; footprint (none) -> kicad-libraries:CON-SENSOR2
- P2: value (none) -> CONN_5; footprint (none) -> kicad-libraries:AKL_5_5
- P3: value (none) -> BOOT; footprint (none) -> kicad-libraries:SolderJumper
- P4: value (none) -> DEBUG; footprint (none) -> kicad-libraries:DEBUG_PAD
- R1: value (none) -> 68.1; footprint (none) -> kicad-libraries:R0603F
- R2: value (none) -> 0; footprint (none) -> kicad-libraries:R0603F
- R3, R4: value (none) -> 10k; footprint (none) -> kicad-libraries:R0603F
- R5, R6: value (none) -> 130k; footprint (none) -> kicad-libraries:R0603F
- R7: value (none) -> 10; footprint (none) -> kicad-libraries:R0603F
- R8: value (none) -> 1k; footprint (none) -> kicad-libraries:R0603F
- RP1: value (none) -> 82; footprint (none) -> kicad-libraries:4X0402
- U1: value (none) -> XMC110024; footprint (none) -> kicad-libraries:QFN24-4x4mm-0.5mm
- U2: value (none) -> TLV272IS; footprint (none) -> kicad-libraries:SOIC8
- U3, U4, U5, U6: value (none) -> DRILL; footprint (none) -> kicad-libraries:DRILL_NP
Other:
- note added: "Copyright Tinkerforge GmbH 2023. This documentation describes Open Hardware and is licensed under the CERN OHL v. 1.1. You may redistribute and modify this documentation under the terms of the CERN OHL v.1.1. (http://ohwr.org/cernohl). This documentation is distributed WITHOUT ANY EXPRESS OR IMPLIED WARRANTY, INCLUDING OF MERCHANTABILITY, SATISFACTORY QUALITY AND FITNESS FOR A PARTICULAR PURPOSE.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"
- note removed: "Copyright Tinkerforge GmbH 2017. This documentation describes Open Hardware and is licensed under the CERN OHL v. 1.1. You may redistribute and modify this documentation under the terms of the CERN OHL v.1.1. (http://ohwr.org/cernohl). This documentation is distributed WITHOUT ANY EXPRESS OR IMPLIED WARRANTY, INCLUDING OF MERCHANTABILITY, SATISFACTORY QUALITY AND FITNESS FOR A PARTICULAR PURPOSE.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"
